Commit message: test with latest platform

File: p3dx_description/urdf/pioneer3dx.xacro (robot description, xacro)
@@ -21,4 +21,9 @@
   <!-- import the pioneer 3dx's wheels -->
   <xacro:include filename="$(find p3dx_description)/urdf/pioneer3dx_wheel.xacro" />
+	<!-- <link name="dummy" />
+	<joint name="dummy_joint" type="fixed">
+		<parent link="dummy"/>
+		<child link="base_link"/>
+	</joint> -->
   <!-- chassis -->
 	<link name="base_link">
